Commit message: Add depth camera integration and pose grasp demo functionality
- Included a depth camera link and joint in the URDF model.
- Added gazebo plugins for the depth camera.
- Enhanced RG2 gripper with movable finger joints.
- Created new launch files for circle stacking and pose grasping demos.
- Implemented interactive prompt for pose grasp demo parameters.
- Developed C++ node for executing pose grasp demo with MoveIt integration.

File: agbot/leaf_manipulation_sim/urdf/fixed_tm5_rg2.urdf.xacro (robot description, xacro)
@@ -5,4 +5,5 @@
   <xacro:include filename="$(find leaf_manipulation_sim)/urdf/parts/rg2_mount.xacro"/>
   <xacro:include filename="$(find leaf_manipulation_sim)/urdf/parts/floor_mount.xacro"/>
+  <xacro:include filename="$(find leaf_manipulation_sim)/urdf/parts/gazebo_plugins.xacro"/>
   <xacro:include filename="$(find leaf_manipulation_sim)/urdf/parts/gazebo_collision_safe.xacro"/>
   <xacro:property name="plate_height" value="0.05"/>
@@ -16,4 +17,40 @@
     <origin xyz="0 0 ${plate_height}" rpy="0 0 0"/>
   </joint>
+  <link name="camera_link">
+    <visual>
+      <geometry>
+        <box size="0.04 0.09 0.03"/>
+      </geometry>
+      <material name="camera_black">
+        <color rgba="0.10 0.10 0.10 1.0"/>
+      </material>
+    </visual>
+    <collision>
+      <geometry>
+        <box size="0.04 0.09 0.03"/>
+      </geometry>
+    </collision>
+    <inertial>
+      <mass value="0.10"/>
+      <inertia ixx="0.0002" ixy="0.0" ixz="0.0" iyy="0.0002" iyz="0.0" izz="0.0002"/>
+    </inertial>
+  </link>
+  <joint name="hand_camera_joint" type="fixed">
+    <parent link="link_6"/>
+    <child link="camera_link"/>
+    <origin xyz="0.0175 0.1243 0.01933" rpy="0.0 -1.5707 -1.5707"/>
+  </joint>
+  <link name="camera_color_optical_frame"/>
+  <joint name="camera_color_optical_joint" type="fixed">
+    <parent link="camera_link"/>
+    <child link="camera_color_optical_frame"/>
+    <origin xyz="0 0 0" rpy="-1.57079632679 0 -1.57079632679"/>
+  </joint>
+  <link name="camera_depth_optical_frame"/>
+  <joint name="camera_depth_optical_joint" type="fixed">
+    <parent link="camera_link"/>
+    <child link="camera_depth_optical_frame"/>
+    <origin xyz="0 0 0" rpy="-1.57079632679 0 -1.57079632679"/>
+  </joint>
   <xacro:rg2_gripper prefix="" parent_link="flange"/>
   <gazebo>
@@ -22,3 +59,7 @@
   <xacro:tm5_gazebo_safe prefix=""/>
   <xacro:rg2_gazebo_safe prefix=""/>
+  <xacro:bench_depth_camera
+      parent_link="camera_link"
+      frame_name="camera_depth_optical_frame"
+      namespace="/camera"/>
 </robot>

File: agbot/leaf_manipulation_sim/urdf/parts/gazebo_plugins.xacro (robot description, xacro)
@@ -48,5 +48,5 @@
     </gazebo>
   </xacro:macro>
-  <xacro:macro name="bench_depth_camera" params="parent_link:='camera_link'">
+  <xacro:macro name="bench_depth_camera" params="parent_link:='camera_link' frame_name:='camera_depth_optical_frame' namespace:='/camera'">
     <gazebo reference="${parent_link}">
       <sensor name="bench_depth_camera" type="depth">
@@ -68,5 +68,5 @@
         <plugin name="bench_depth_camera_plugin" filename="libgazebo_ros_camera.so">
           <ros>
-            <namespace>/camera</namespace>
+            <namespace>${namespace}</namespace>
             <remapping>~/image_raw:=color/image_raw</remapping>
             <remapping>~/camera_info:=color/camera_info</remapping>
@@ -75,5 +75,5 @@
             <remapping>~/depth/points:=depth/color/points</remapping>
           </ros>
-          <frame_name>${parent_link}</frame_name>
+          <frame_name>${frame_name}</frame_name>
         </plugin>
       </sensor>

File: agbot/leaf_manipulation_sim/urdf/parts/rg2_mount.xacro (robot description, xacro)
@@ -3,10 +3,55 @@
   <xacro:include filename="$(find onrobot_rg_description)/urdf/onrobot_rg2_model_macro.xacro"/>
   <!-- Visual-only RG2 mount: no transmission (avoids ros_control deps in stage 2) -->
+  <xacro:macro name="movable_inner_knuckle_joint" params="prefix fingerprefix reflect">
+    <joint name="${prefix}${fingerprefix}_inner_knuckle_joint" type="revolute">
+      <origin xyz="0 ${reflect * -0.007678} 0.1422970" rpy="0 0 ${(reflect - 1) * pi / 2}" />
+      <parent link="${prefix}onrobot_rg2_base_link" />
+      <child link="${prefix}${fingerprefix}_inner_knuckle" />
+      <axis xyz="1 0 0" />
+      <limit lower="-0.785398" upper="0.785398" velocity="100.0" effort="1000" />
+      <mimic joint="${prefix}finger_joint" multiplier="-1" offset="0" />
+    </joint>
+  </xacro:macro>
+  <xacro:macro name="movable_inner_finger_joint" params="prefix fingerprefix">
+    <joint name="${prefix}${fingerprefix}_inner_finger_joint" type="revolute">
+      <origin xyz="0 ${-(0.056770-0.017178)} ${0.163974-0.125797}" rpy="0 0 0" />
+      <parent link="${prefix}${fingerprefix}_outer_knuckle" />
+      <child link="${prefix}${fingerprefix}_inner_finger" />
+      <axis xyz="1 0 0" />
+      <limit lower="-0.872665" upper="0.872665" velocity="100.0" effort="1000" />
+      <mimic joint="${prefix}finger_joint" multiplier="1" offset="0" />
+    </joint>
+  </xacro:macro>
+  <xacro:macro name="movable_finger_joints" params="prefix fingerprefix reflect">
+    <xacro:movable_inner_knuckle_joint prefix="${prefix}" fingerprefix="${fingerprefix}" reflect="${reflect}"/>
+    <xacro:movable_inner_finger_joint prefix="${prefix}" fingerprefix="${fingerprefix}"/>
+  </xacro:macro>
+  <xacro:macro name="movable_finger_joint" params="prefix">
+    <joint name="${prefix}finger_joint" type="revolute">
+      <origin xyz="0 -0.017178 0.125797" rpy="0 0 0" />
+      <parent link="${prefix}onrobot_rg2_base_link" />
+      <child link="${prefix}left_outer_knuckle" />
+      <axis xyz="-1 0 0" />
+      <limit lower="-0.558505" upper="0.785398" velocity="100.0" effort="1000" />
+    </joint>
+    <xacro:movable_finger_joints prefix="${prefix}" fingerprefix="left" reflect="1.0"/>
+  </xacro:macro>
+  <xacro:macro name="movable_right_outer_knuckle_joint" params="prefix">
+    <joint name="${prefix}right_outer_knuckle_joint" type="revolute">
+      <origin xyz="0 0.017178 0.125797" rpy="0 0 ${pi}" />
+      <parent link="${prefix}onrobot_rg2_base_link" />
+      <child link="${prefix}right_outer_knuckle" />
+      <axis xyz="1 0 0" />
+      <limit lower="-0.785398" upper="0.785398" velocity="100.0" effort="1000" />
+      <mimic joint="${prefix}finger_joint" multiplier="-1" offset="0" />
+    </joint>
+    <xacro:movable_finger_joints prefix="${prefix}" fingerprefix="right" reflect="-1.0"/>
+  </xacro:macro>
   <xacro:macro name="rg2_gripper" params="prefix:='' parent_link:='flange'">
     <xacro:onrobot_rg2_base_link prefix="${prefix}"/>
     <xacro:finger_links prefix="${prefix}" fingerprefix="left"/>
     <xacro:finger_links prefix="${prefix}" fingerprefix="right"/>
-    <xacro:finger_joint prefix="${prefix}"/>
-    <xacro:right_outer_knuckle_joint prefix="${prefix}"/>
+    <xacro:movable_finger_joint prefix="${prefix}"/>
+    <xacro:movable_right_outer_knuckle_joint prefix="${prefix}"/>
     <joint name="${prefix}rg2_mount_joint" type="fixed">
       <parent link="${parent_link}"/>

Commit message: Add calibration floor model for RGBD camera and scale checks
- Introduced model.config for the Metric Calibration Floor with versioning and description.
- Created model.sdf defining a static calibration floor with collision and visual properties, including friction settings and material references.

File: agbot/leaf_manipulation_sim/urdf/fixed_tm5_rg2.urdf.xacro (robot description, xacro)
@@ -17,28 +17,33 @@
     <origin xyz="0 0 ${plate_height}" rpy="0 0 0"/>
   </joint>
+  <xacro:rg2_gripper prefix="" parent_link="flange"/>
+  <!-- Official Intel RealSense D435 visual; Gazebo's sanitized copy uses a box. -->
   <link name="camera_link">
     <visual>
+      <origin xyz="0.0043 -0.0175 0" rpy="1.57079632679 0 1.57079632679"/>
       <geometry>
-        <box size="0.04 0.09 0.03"/>
+        <mesh filename="package://realsense2_description/meshes/d435.dae"/>
       </geometry>
-      <material name="camera_black">
-        <color rgba="0.10 0.10 0.10 1.0"/>
-      </material>
     </visual>
     <collision>
+      <origin xyz="0 -0.0175 0" rpy="0 0 0"/>
       <geometry>
-        <box size="0.04 0.09 0.03"/>
+        <box size="0.02505 0.090 0.025"/>
       </geometry>
     </collision>
     <inertial>
-      <mass value="0.10"/>
-      <inertia ixx="0.0002" ixy="0.0" ixz="0.0" iyy="0.0002" iyz="0.0" izz="0.0002"/>
+      <mass value="0.072"/>
+      <inertia ixx="0.003881243" ixy="0" ixz="0" iyy="0.000498940" iyz="0" izz="0.003879257"/>
     </inertial>
   </link>
+  <!-- RoMu4o eye-in-hand camera pose from the original TM model. -->
   <joint name="hand_camera_joint" type="fixed">
     <parent link="link_6"/>
     <child link="camera_link"/>
-    <origin xyz="0.0175 0.1243 0.01933" rpy="0.0 -1.5707 -1.5707"/>
+    <origin xyz="0.0175 0.1243 0.01933" rpy="0 -1.5707 -1.5707"/>
   </joint>
+  <gazebo reference="hand_camera_joint">
+    <preserveFixedJoint>true</preserveFixedJoint>
+  </gazebo>
   <link name="camera_color_optical_frame"/>
   <joint name="camera_color_optical_joint" type="fixed">
@@ -53,5 +58,4 @@
     <origin xyz="0 0 0" rpy="-1.57079632679 0 -1.57079632679"/>
   </joint>
-  <xacro:rg2_gripper prefix="" parent_link="flange"/>
   <gazebo>
     <static>true</static>
@@ -59,7 +63,3 @@
   <xacro:tm5_gazebo_safe prefix=""/>
   <xacro:rg2_gazebo_safe prefix=""/>
-  <xacro:bench_depth_camera
-      parent_link="camera_link"
-      frame_name="camera_depth_optical_frame"
-      namespace="/camera"/>
 </robot>

Commit message: Add simple potted plant model configuration and SDF definition
- Created model.config for the Simple Potted Plant with metadata including name, version, author, and description.
- Added model.sdf file defining the visual and collision properties of the potted plant, including mesh and simplified collision geometry for robust contact handling.

File: agbot/leaf_manipulation_sim/urdf/fixed_tm5_rg2.urdf.xacro (robot description, xacro)
@@ -18,5 +18,5 @@
   </joint>
   <xacro:rg2_gripper prefix="" parent_link="flange"/>
-  <!-- Official Intel RealSense D435 visual; Gazebo's sanitized copy uses a box. -->
+  <!-- Official Intel RealSense D435 visual, shared by RViz and Gazebo. -->
   <link name="camera_link">
     <visual>

File: agbot/leaf_manipulation_sim/urdf/leaf_arm.sim.urdf.xacro (robot description, xacro)
@@ -3,4 +3,5 @@
   <xacro:include filename="$(find tm_description)/xacro/macro.materials.xacro"/>
   <xacro:include filename="$(find tm_description)/xacro/macro.tm5-900-nominal.urdf.xacro"/>
+  <xacro:include filename="$(find realsense2_description)/urdf/_d435.urdf.xacro"/>
   <xacro:include filename="$(find leaf_manipulation_sim)/urdf/parts/fixed_mount.xacro"/>
   <xacro:include filename="$(find leaf_manipulation_sim)/urdf/parts/rg2_mount.xacro"/>
@@ -8,9 +9,8 @@
   <xacro:include filename="$(find leaf_manipulation_sim)/urdf/parts/gazebo_collision_safe.xacro"/>
   <link name="world"/>
-  <xacro:fixed_pedestal height="0.75" width="0.45" depth="0.45"/>
-  <xacro:bench_camera parent_link="pedestal_link"/>
+  <xacro:fixed_pedestal height="0.05" width="0.50" depth="0.50"/>
   <xacro:property name="arm_mount_x" value="0.0"/>
   <xacro:property name="arm_mount_y" value="0.0"/>
-  <xacro:property name="arm_mount_z" value="0.40"/>
+  <xacro:property name="arm_mount_z" value="0.025"/>
   <xacro:property name="arm_mount_roll" value="0.0"/>
   <xacro:property name="arm_mount_pitch" value="0.0"/>
@@ -25,4 +25,29 @@
   </joint>
   <xacro:rg2_gripper prefix="" parent_link="flange"/>
+  <!-- Native TMvision optical pose from the official modified TM5-900 model. -->
+  <link name="tmvision_camera_frame"/>
+  <joint name="tmvision_camera_joint" type="fixed">
+    <parent link="link_6"/>
+    <child link="tmvision_camera_frame"/>
+    <origin xyz="0.0175 0.1243 0.01933" rpy="0 -1.5707 -1.5707"/>
+  </joint>
+  <!--
+    Align the D435 with TMvision and place its depth-camera frame 15 mm in
+    front of the native lens.  The offset below compensates for the official
+    D435 model's bottom-screw-to-camera-frame transform, leaving the detailed
+    D435 body about 2.5 mm in front of the TMvision lens surface.
+  -->
+  <xacro:sensor_d435
+    parent="link_6"
+    name="camera"
+    use_nominal_extrinsics="true"
+    add_plug="false"
+    use_mesh="true">
+    <!-- Equivalent to xyz="0.0044 -0.0175 -0.0125" in TMvision frame. -->
+    <origin xyz="0.0 0.1118 0.02373" rpy="0 -1.5707 -1.5707"/>
+  </xacro:sensor_d435>
+  <gazebo reference="camera_joint">
+    <preserveFixedJoint>true</preserveFixedJoint>
+  </gazebo>
   <xacro:tm5_gazebo_safe prefix=""/>
   <xacro:rg2_gazebo_safe prefix=""/>
@@ -41,5 +66,6 @@
   </ros2_control>
   <xacro:gazebo_ros2_control_plugin/>
-  <xacro:bench_depth_camera parent_link="camera_link"/>
+  <!-- Gazebo reduces camera_link into this preserved mounting frame. -->
+  <xacro:d435_depth_camera parent_link="camera_bottom_screw_frame"/>
   <gazebo reference="link_1"><selfCollide>true</selfCollide></gazebo>
   <gazebo reference="link_2"><selfCollide>true</selfCollide></gazebo>

File: agbot/leaf_manipulation_sim/urdf/parts/gazebo_plugins.xacro (robot description, xacro)
@@ -47,7 +47,7 @@
     </gazebo>
   </xacro:macro>
-  <xacro:macro name="bench_depth_camera" params="parent_link:='camera_link' frame_name:='camera_depth_optical_frame' namespace:='/camera'">
+  <xacro:macro name="d435_depth_camera" params="parent_link:='camera_link' frame_name:='camera_depth_optical_frame' namespace:='/camera'">
     <gazebo reference="${parent_link}">
-      <sensor name="bench_depth_camera" type="depth">
+      <sensor name="d435_depth_camera" type="depth">
         <always_on>true</always_on>
         <update_rate>10.0</update_rate>
@@ -65,12 +65,12 @@
           </clip>
         </camera>
-        <plugin name="bench_depth_camera_plugin" filename="libgazebo_ros_camera.so">
+        <plugin name="d435_plugin" filename="libgazebo_ros_camera.so">
           <ros>
             <namespace>${namespace}</namespace>
-            <remapping>bench_depth_camera/image_raw:=color/image_raw</remapping>
-            <remapping>bench_depth_camera/camera_info:=color/camera_info</remapping>
-            <remapping>bench_depth_camera/depth/image_raw:=depth/image_raw</remapping>
-            <remapping>bench_depth_camera/depth/camera_info:=depth/camera_info</remapping>
-            <remapping>bench_depth_camera/points:=depth/color/points</remapping>
+            <remapping>d435_depth_camera/image_raw:=color/image_raw</remapping>
+            <remapping>d435_depth_camera/camera_info:=color/camera_info</remapping>
+            <remapping>d435_depth_camera/depth/image_raw:=depth/image_raw</remapping>
+            <remapping>d435_depth_camera/depth/camera_info:=depth/camera_info</remapping>
+            <remapping>d435_depth_camera/points:=depth/color/points</remapping>
           </ros>
           <frame_name>${frame_name}</frame_name>
