Commit message: Refactor leaf manipulation simulation for improved functionality and integration
- Updated URDF paths and configurations to use the new leaf_arm.sim.urdf model.
- Enhanced launch files to include GUI options and improved parameter handling.
- Replaced static joint state publisher with dynamic command publishers for arm and gripper.
- Integrated initial controller commands to set the robot to a ready pose.
- Modified MoveIt configurations to accommodate new robot structure and joint names.
- Improved RViz configuration to visualize RGB and depth images from the camera.
- Updated Gazebo plugins to use ros2_control for better control interface.
- Added support for new camera frames in the URDF.
- Enhanced world file to include camera settings for better simulation views.
- Fixed various issues related to joint state publishing and controller readiness checks.

File: agbot/leaf_manipulation_sim/urdf/leaf_arm.sim.urdf.xacro (robot description, xacro)
@@ -1,7 +1,6 @@
 <?xml version="1.0"?>
-<robot name="leaf_manipulation_sim" xmlns:xacro="http://www.ros.org/wiki/xacro">
+<robot name="tm5-900" xmlns:xacro="http://www.ros.org/wiki/xacro">
   <xacro:include filename="$(find tm_description)/xacro/macro.materials.xacro"/>
   <xacro:include filename="$(find tm_description)/xacro/macro.tm5-900-nominal.urdf.xacro"/>
-  <xacro:include filename="$(find tm_description)/xacro/macro.transmission.xacro"/>
   <xacro:include filename="$(find leaf_manipulation_sim)/urdf/parts/fixed_mount.xacro"/>
   <xacro:include filename="$(find leaf_manipulation_sim)/urdf/parts/rg2_mount.xacro"/>
@@ -19,5 +18,4 @@
   <xacro:tmr_materials/>
   <xacro:tm5-900 ns="" prefix="" color="white" format="stl"/>
-  <xacro:tmr_transmission prefix="" hw_iface="hardware_interface/PositionJointInterface"/>
   <joint name="pedestal_to_arm_base" type="fixed">
     <parent link="pedestal_link"/>
@@ -30,5 +28,17 @@
   <xacro:rg2_gazebo_safe prefix=""/>
   <xacro:rg2_mimic_plugins prefix=""/>
-  <xacro:gazebo_ros_control_plugin/>
+  <ros2_control name="GazeboSystem" type="system">
+    <hardware>
+      <plugin>gazebo_ros2_control/GazeboSystem</plugin>
+    </hardware>
+    <joint name="joint_1"><command_interface name="position"/><state_interface name="position"/><state_interface name="velocity"/></joint>
+    <joint name="joint_2"><command_interface name="position"/><state_interface name="position"/><state_interface name="velocity"/></joint>
+    <joint name="joint_3"><command_interface name="position"/><state_interface name="position"/><state_interface name="velocity"/></joint>
+    <joint name="joint_4"><command_interface name="position"/><state_interface name="position"/><state_interface name="velocity"/></joint>
+    <joint name="joint_5"><command_interface name="position"/><state_interface name="position"/><state_interface name="velocity"/></joint>
+    <joint name="joint_6"><command_interface name="position"/><state_interface name="position"/><state_interface name="velocity"/></joint>
+    <joint name="finger_joint"><command_interface name="position"/><state_interface name="position"/><state_interface name="velocity"/></joint>
+  </ros2_control>
+  <xacro:gazebo_ros2_control_plugin/>
   <xacro:bench_depth_camera parent_link="camera_link"/>
   <gazebo reference="link_1"><selfCollide>true</selfCollide></gazebo>

File: agbot/leaf_manipulation_sim/urdf/parts/fixed_mount.xacro (robot description, xacro)
@@ -57,4 +57,16 @@
       <origin xyz="0.30 0.0 0.45" rpy="0 0.35 0"/>
     </joint>
+    <link name="camera_color_optical_frame"/>
+    <joint name="camera_color_optical_joint" type="fixed">
+      <parent link="camera_link"/>
+      <child link="camera_color_optical_frame"/>
+      <origin xyz="0 0 0" rpy="-1.57079632679 0 -1.57079632679"/>
+    </joint>
+    <link name="camera_depth_optical_frame"/>
+    <joint name="camera_depth_optical_joint" type="fixed">
+      <parent link="camera_link"/>
+      <child link="camera_depth_optical_frame"/>
+      <origin xyz="0 0 0" rpy="-1.57079632679 0 -1.57079632679"/>
+    </joint>
   </xacro:macro>
 </robot>

File: agbot/leaf_manipulation_sim/urdf/parts/gazebo_plugins.xacro (robot description, xacro)
@@ -40,9 +40,8 @@
     </gazebo>
   </xacro:macro>
-  <xacro:macro name="gazebo_ros_control_plugin">
+  <xacro:macro name="gazebo_ros2_control_plugin">
     <gazebo>
-      <plugin name="gazebo_ros_control" filename="libgazebo_ros_control.so">
-        <robotNamespace>/</robotNamespace>
-        <robotSimType>gazebo_ros_control/DefaultRobotHWSim</robotSimType>
+      <plugin name="gazebo_ros2_control" filename="libgazebo_ros2_control.so">
+        <parameters>$(find leaf_manipulation_sim)/config/arm_controllers.yaml</parameters>
       </plugin>
     </gazebo>
@@ -69,9 +68,9 @@
           <ros>
             <namespace>${namespace}</namespace>
-            <remapping>~/image_raw:=color/image_raw</remapping>
-            <remapping>~/camera_info:=color/camera_info</remapping>
-            <remapping>~/depth/image_raw:=depth/image_raw</remapping>
-            <remapping>~/depth/camera_info:=depth/camera_info</remapping>
-            <remapping>~/depth/points:=depth/color/points</remapping>
+            <remapping>bench_depth_camera/image_raw:=color/image_raw</remapping>
+            <remapping>bench_depth_camera/camera_info:=color/camera_info</remapping>
+            <remapping>bench_depth_camera/depth/image_raw:=depth/image_raw</remapping>
+            <remapping>bench_depth_camera/depth/camera_info:=depth/camera_info</remapping>
+            <remapping>bench_depth_camera/points:=depth/color/points</remapping>
           </ros>
           <frame_name>${frame_name}</frame_name>

Commit message: 更改gazebo版本

File: agbot/leaf_manipulation_sim/urdf/leaf_arm.sim.urdf.xacro (robot description, xacro)
@@ -6,5 +6,5 @@
   <xacro:include filename="$(find leaf_manipulation_sim)/urdf/parts/fixed_mount.xacro"/>
   <xacro:include filename="$(find leaf_manipulation_sim)/urdf/parts/rg2_mount.xacro"/>
-  <xacro:include filename="$(find leaf_manipulation_sim)/urdf/parts/gazebo_plugins.xacro"/>
+  <xacro:include filename="$(find leaf_manipulation_sim)/urdf/parts/gz_plugins.xacro"/>
   <xacro:include filename="$(find leaf_manipulation_sim)/urdf/parts/gazebo_collision_safe.xacro"/>
   <link name="world"/>
@@ -24,5 +24,5 @@
             rpy="${arm_mount_roll} ${arm_mount_pitch} ${arm_mount_yaw}"/>
   </joint>
-  <xacro:rg2_gripper prefix="" parent_link="flange"/>
+  <xacro:rg2_gripper prefix="" parent_link="flange" use_urdf_mimic="false"/>
   <!-- Native TMvision optical pose from the official modified TM5-900 model. -->
   <link name="tmvision_camera_frame"/>
@@ -52,8 +52,7 @@
   <xacro:tm5_gazebo_safe prefix=""/>
   <xacro:rg2_gazebo_safe prefix=""/>
-  <xacro:rg2_mimic_plugins prefix=""/>
-  <ros2_control name="GazeboSystem" type="system">
+  <ros2_control name="GazeboSimSystem" type="system">
     <hardware>
-      <plugin>gazebo_ros2_control/GazeboSystem</plugin>
+      <plugin>gz_ros2_control/GazeboSimSystem</plugin>
     </hardware>
     <joint name="joint_1"><command_interface name="position"/><state_interface name="position"/><state_interface name="velocity"/></joint>
@@ -64,8 +63,13 @@
     <joint name="joint_6"><command_interface name="position"/><state_interface name="position"/><state_interface name="velocity"/></joint>
     <joint name="finger_joint"><command_interface name="position"/><state_interface name="position"/><state_interface name="velocity"/></joint>
+    <joint name="left_inner_knuckle_joint"><command_interface name="position"/><state_interface name="position"/><state_interface name="velocity"/></joint>
+    <joint name="left_inner_finger_joint"><command_interface name="position"/><state_interface name="position"/><state_interface name="velocity"/></joint>
+    <joint name="right_outer_knuckle_joint"><command_interface name="position"/><state_interface name="position"/><state_interface name="velocity"/></joint>
+    <joint name="right_inner_knuckle_joint"><command_interface name="position"/><state_interface name="position"/><state_interface name="velocity"/></joint>
+    <joint name="right_inner_finger_joint"><command_interface name="position"/><state_interface name="position"/><state_interface name="velocity"/></joint>
   </ros2_control>
-  <xacro:gazebo_ros2_control_plugin/>
+  <xacro:gz_ros2_control_plugin/>
   <!-- Gazebo reduces camera_link into this preserved mounting frame. -->
-  <xacro:d435_depth_camera parent_link="camera_bottom_screw_frame"/>
+  <xacro:d435_gz_rgbd_camera parent_link="camera_bottom_screw_frame"/>
   <gazebo reference="link_1"><selfCollide>true</selfCollide></gazebo>
   <gazebo reference="link_2"><selfCollide>true</selfCollide></gazebo>

File: agbot/leaf_manipulation_sim/urdf/parts/rg2_mount.xacro (robot description, xacro)
@@ -3,5 +3,5 @@
   <xacro:include filename="$(find onrobot_rg_description)/urdf/onrobot_rg2_model_macro.xacro"/>
   <!-- Visual-only RG2 mount: no transmission (avoids ros_control deps in stage 2) -->
-  <xacro:macro name="movable_inner_knuckle_joint" params="prefix fingerprefix reflect">
+  <xacro:macro name="movable_inner_knuckle_joint" params="prefix fingerprefix reflect use_urdf_mimic">
     <joint name="${prefix}${fingerprefix}_inner_knuckle_joint" type="revolute">
       <origin xyz="0 ${reflect * -0.007678} 0.1422970" rpy="0 0 ${(reflect - 1) * pi / 2}" />
@@ -10,8 +10,10 @@
       <axis xyz="1 0 0" />
       <limit lower="-0.785398" upper="0.785398" velocity="100.0" effort="1000" />
-      <mimic joint="${prefix}finger_joint" multiplier="-1" offset="0" />
+      <xacro:if value="${use_urdf_mimic}">
+        <mimic joint="${prefix}finger_joint" multiplier="-1" offset="0" />
+      </xacro:if>
     </joint>
   </xacro:macro>
-  <xacro:macro name="movable_inner_finger_joint" params="prefix fingerprefix">
+  <xacro:macro name="movable_inner_finger_joint" params="prefix fingerprefix use_urdf_mimic">
     <joint name="${prefix}${fingerprefix}_inner_finger_joint" type="revolute">
       <origin xyz="0 ${-(0.056770-0.017178)} ${0.163974-0.125797}" rpy="0 0 0" />
@@ -20,12 +22,14 @@
       <axis xyz="1 0 0" />
       <limit lower="-0.872665" upper="0.872665" velocity="100.0" effort="1000" />
-      <mimic joint="${prefix}finger_joint" multiplier="1" offset="0" />
+      <xacro:if value="${use_urdf_mimic}">
+        <mimic joint="${prefix}finger_joint" multiplier="1" offset="0" />
+      </xacro:if>
     </joint>
   </xacro:macro>
-  <xacro:macro name="movable_finger_joints" params="prefix fingerprefix reflect">
-    <xacro:movable_inner_knuckle_joint prefix="${prefix}" fingerprefix="${fingerprefix}" reflect="${reflect}"/>
-    <xacro:movable_inner_finger_joint prefix="${prefix}" fingerprefix="${fingerprefix}"/>
+  <xacro:macro name="movable_finger_joints" params="prefix fingerprefix reflect use_urdf_mimic">
+    <xacro:movable_inner_knuckle_joint prefix="${prefix}" fingerprefix="${fingerprefix}" reflect="${reflect}" use_urdf_mimic="${use_urdf_mimic}"/>
+    <xacro:movable_inner_finger_joint prefix="${prefix}" fingerprefix="${fingerprefix}" use_urdf_mimic="${use_urdf_mimic}"/>
   </xacro:macro>
-  <xacro:macro name="movable_finger_joint" params="prefix">
+  <xacro:macro name="movable_finger_joint" params="prefix use_urdf_mimic">
     <joint name="${prefix}finger_joint" type="revolute">
       <origin xyz="0 -0.017178 0.125797" rpy="0 0 0" />
@@ -35,7 +39,7 @@
       <limit lower="-0.558505" upper="0.785398" velocity="100.0" effort="1000" />
     </joint>
-    <xacro:movable_finger_joints prefix="${prefix}" fingerprefix="left" reflect="1.0"/>
+    <xacro:movable_finger_joints prefix="${prefix}" fingerprefix="left" reflect="1.0" use_urdf_mimic="${use_urdf_mimic}"/>
   </xacro:macro>
-  <xacro:macro name="movable_right_outer_knuckle_joint" params="prefix">
+  <xacro:macro name="movable_right_outer_knuckle_joint" params="prefix use_urdf_mimic">
     <joint name="${prefix}right_outer_knuckle_joint" type="revolute">
       <origin xyz="0 0.017178 0.125797" rpy="0 0 ${pi}" />
@@ -44,14 +48,16 @@
       <axis xyz="1 0 0" />
       <limit lower="-0.785398" upper="0.785398" velocity="100.0" effort="1000" />
-      <mimic joint="${prefix}finger_joint" multiplier="-1" offset="0" />
+      <xacro:if value="${use_urdf_mimic}">
+        <mimic joint="${prefix}finger_joint" multiplier="-1" offset="0" />
+      </xacro:if>
     </joint>
-    <xacro:movable_finger_joints prefix="${prefix}" fingerprefix="right" reflect="-1.0"/>
+    <xacro:movable_finger_joints prefix="${prefix}" fingerprefix="right" reflect="-1.0" use_urdf_mimic="${use_urdf_mimic}"/>
   </xacro:macro>
-  <xacro:macro name="rg2_gripper" params="prefix:='' parent_link:='flange'">
+  <xacro:macro name="rg2_gripper" params="prefix:='' parent_link:='flange' use_urdf_mimic:='true'">
     <xacro:onrobot_rg2_base_link prefix="${prefix}"/>
     <xacro:finger_links prefix="${prefix}" fingerprefix="left"/>
     <xacro:finger_links prefix="${prefix}" fingerprefix="right"/>
-    <xacro:movable_finger_joint prefix="${prefix}"/>
-    <xacro:movable_right_outer_knuckle_joint prefix="${prefix}"/>
+    <xacro:movable_finger_joint prefix="${prefix}" use_urdf_mimic="${use_urdf_mimic}"/>
+    <xacro:movable_right_outer_knuckle_joint prefix="${prefix}" use_urdf_mimic="${use_urdf_mimic}"/>
     <joint name="${prefix}rg2_mount_joint" type="fixed">
       <parent link="${parent_link}"/>

Commit message: Add Gazebo plugins for ROS2 control and RGB-D camera integration
- Introduced gz_ros2_control_plugin macro for integrating ROS2 control with Gazebo.
- Added d435_gz_rgbd_camera macro to configure RGB-D camera settings and parameters.
- The new xacro file enhances simulation capabilities for the leaf manipulation project.

File: agbot/leaf_manipulation_sim/urdf/leaf_arm.sim.urdf.xacro (robot description, xacro)
@@ -33,8 +33,9 @@
   </joint>
   <!--
-    Align the D435 with TMvision and place its depth-camera frame 15 mm in
-    front of the native lens.  The offset below compensates for the official
-    D435 model's bottom-screw-to-camera-frame transform, leaving the detailed
-    D435 body about 2.5 mm in front of the TMvision lens surface.
+    Mount the D435 sideways and centre its body on the TMvision side face.
+    The D435 macro is anchored at its bottom screw rather than at the body
+    centre, so the 12.5 mm Y offset below keeps the body centred while applying
+    the 90 degree in-plane rotation.  Its optical +X axis still points downward
+    in the ready1 arm pose.
   -->
   <xacro:sensor_d435
@@ -44,6 +45,6 @@
     add_plug="false"
     use_mesh="true">
-    <!-- Equivalent to xyz="0.0044 -0.0175 -0.0125" in TMvision frame. -->
-    <origin xyz="0.0 0.1118 0.02373" rpy="0 -1.5707 -1.5707"/>
+    <origin xyz="0.0 0.1243 0.02373"
+            rpy="1.5708 -1.5708 0.0"/>
   </xacro:sensor_d435>
   <gazebo reference="camera_joint">

File: agbot/leaf_manipulation_sim/urdf/parts/gz_plugins.xacro (robot description, xacro)
@@ -16,4 +16,7 @@
     <gazebo reference="${parent_link}">
       <sensor name="d435_depth_camera" type="rgbd_camera">
+        <!-- Flip the rendered image about the optical axis without moving the
+             D435 body, collision geometry, or ROS optical frames. -->
+        <pose>0 0 0 3.141592653589793 0 0</pose>
         <always_on>true</always_on>
         <update_rate>10.0</update_rate>
