Commit message: Add Pro450 simulation files and configurations
- Created RViz configuration file for Pro450 simulation.
- Added scripts for generating scaled plant models and publishing plant markers.
- Implemented a leaf pipeline script for running the Pro450/F100 profile.
- Introduced a world file for the Pro450 leaf bench simulation environment.
- Added necessary Python scripts for marker publishing and model generation.

File: agbot/pro450_description/urdf/pro450_f100.urdf.xacro (robot description, xacro)
@@ -1,9 +1,30 @@
 <?xml version="1.0"?>
 <robot xmlns:xacro="http://www.ros.org/wiki/xacro" name="mycobot_pro_450_f100">
+  <xacro:arg name="use_gz_control" default="false"/>
+  <xacro:arg name="collision_mesh_scale" default="1.0"/>
   <!-- Vendor geometry and kinematic chain imported from Elephant Robotics
        mycobot_ros2 Humble commit 3999e2c.  The D435 transform deliberately
        matches the existing TM5 leaf-simulation description. -->
   <xacro:include filename="$(find realsense2_description)/urdf/_d435.urdf.xacro"/>
+  <xacro:include filename="$(find pro450_description)/urdf/pro450_gz_plugins.xacro"/>
 <xacro:property name="width" value=".2" />
+  <!-- Keep the same floor installation datum as the previous TM5 environment. -->
+  <xacro:property name="mount_plate_height" value="0.05"/>
+  <link name="base_root"/>
+  <link name="mount_plate_link">
+    <visual>
+      <origin xyz="0 0 ${mount_plate_height / 2.0}" rpy="0 0 0"/>
+      <geometry><box size="0.50 0.50 ${mount_plate_height}"/></geometry>
+      <material name="mount_plate_gray"><color rgba="0.55 0.55 0.58 1.0"/></material>
+    </visual>
+    <collision>
+      <origin xyz="0 0 ${mount_plate_height / 2.0}" rpy="0 0 0"/>
+      <geometry><box size="0.50 0.50 ${mount_plate_height}"/></geometry>
+    </collision>
+    <inertial><mass value="5.0"/><inertia ixx="0.1" ixy="0" ixz="0" iyy="0.1" iyz="0" izz="0.1"/></inertial>
+  </link>
+  <joint name="root_to_plate" type="fixed">
+    <parent link="base_root"/><child link="mount_plate_link"/><origin xyz="0 0 0" rpy="0 0 0"/>
+  </joint>
   <link name="base">
     <visual>
@@ -15,5 +36,6 @@
     <collision>
       <geometry>
-       <mesh filename="package://pro450_description/meshes/PRO450_J1.dae"/>
+       <mesh filename="package://pro450_description/meshes/PRO450_J1.dae"
+             scale="$(arg collision_mesh_scale) $(arg collision_mesh_scale) $(arg collision_mesh_scale)"/>
         </geometry>
         <origin xyz = "-0.108 -0.003 0 " rpy = " 0 0 -1.5708"/>
@@ -29,9 +51,14 @@
     <collision>
      <geometry>
-       <mesh filename="package://pro450_description/meshes/PRO450_J2.dae"/>
+       <mesh filename="package://pro450_description/meshes/PRO450_J2.dae"
+             scale="$(arg collision_mesh_scale) $(arg collision_mesh_scale) $(arg collision_mesh_scale)"/>
       </geometry>
       <origin xyz = "0.0015 -0.0392 0.0 " rpy = " -1.5708 0 -3.14159 "/>
     </collision>
   </link>
+  <joint name="plate_to_arm_base" type="fixed">
+    <parent link="mount_plate_link"/><child link="base"/>
+    <origin xyz="0 0 ${mount_plate_height}" rpy="0 0 0"/>
+  </joint>
   <link name="link2">
     <visual>
@@ -43,5 +70,6 @@
     <collision>
       <geometry>
-       <mesh filename="package://pro450_description/meshes/PRO450_J3.dae"/>
+       <mesh filename="package://pro450_description/meshes/PRO450_J3.dae"
+             scale="$(arg collision_mesh_scale) $(arg collision_mesh_scale) $(arg collision_mesh_scale)"/>
       </geometry>
       <origin xyz = "0.0598  0.005 -0.203 " rpy = " 0 0 1.5708"/>
@@ -57,5 +85,6 @@
     <collision>
       <geometry>
-       <mesh filename="package://pro450_description/meshes/PRO450_J4.dae"/>
+       <mesh filename="package://pro450_description/meshes/PRO450_J4.dae"
+             scale="$(arg collision_mesh_scale) $(arg collision_mesh_scale) $(arg collision_mesh_scale)"/>
       </geometry>
       <origin xyz = "0.07 0.005 -0.383" rpy = " 0 0 1.5708"/>
@@ -71,5 +100,6 @@
     <collision>
        <geometry>
-       <mesh filename="package://pro450_description/meshes/PRO450_J5.dae"/>
+       <mesh filename="package://pro450_description/meshes/PRO450_J5.dae"
+             scale="$(arg collision_mesh_scale) $(arg collision_mesh_scale) $(arg collision_mesh_scale)"/>
       </geometry>
       <origin xyz = "-0.014 0 0.0 " rpy = " 0 -1.5708 0"/>
@@ -85,5 +115,6 @@
     <collision>
       <geometry>
-       <mesh filename="package://pro450_description/meshes/PRO450_J6.dae"/>
+       <mesh filename="package://pro450_description/meshes/PRO450_J6.dae"
+             scale="$(arg collision_mesh_scale) $(arg collision_mesh_scale) $(arg collision_mesh_scale)"/>
       </geometry>
     <origin xyz = "0.004 -0.024 -0.655 " rpy = " 0 0 0"/>
@@ -99,5 +130,6 @@
     <collision>
       <geometry>
-       <mesh filename="package://pro450_description/meshes/PRO450_J6_end.dae"/>
+       <mesh filename="package://pro450_description/meshes/PRO450_J6_end.dae"
+             scale="$(arg collision_mesh_scale) $(arg collision_mesh_scale) $(arg collision_mesh_scale)"/>
       </geometry>
     <origin xyz = "0 0 0 " rpy = " 3.14159 0 0"/>
@@ -113,5 +145,6 @@
     <collision>
       <geometry>
-       <mesh filename="package://pro450_description/meshes/mygripper_f100_connection.dae"/>
+       <mesh filename="package://pro450_description/meshes/mygripper_f100_connection.dae"
+             scale="$(arg collision_mesh_scale) $(arg collision_mesh_scale) $(arg collision_mesh_scale)"/>
       </geometry>
     <origin xyz = "-0.03 0.014 0 " rpy = " 0  0 -1.5708"/>
@@ -127,5 +160,6 @@
     <collision>
       <geometry>
-       <mesh filename="package://pro450_description/meshes/pro_gripper_base.dae"/>
+       <mesh filename="package://pro450_description/meshes/pro_gripper_base.dae"
+             scale="$(arg collision_mesh_scale) $(arg collision_mesh_scale) $(arg collision_mesh_scale)"/>
       </geometry>
     <origin xyz = "-0.107 0.012 0.0 " rpy = " 1.5708  0 1.5708"/>
@@ -142,5 +176,6 @@
     <collision>
       <geometry>
-       <mesh filename="package://pro450_description/meshes/pro_gripper_left1.dae"/>
+       <mesh filename="package://pro450_description/meshes/pro_gripper_left1.dae"
+             scale="$(arg collision_mesh_scale) $(arg collision_mesh_scale) $(arg collision_mesh_scale)"/>
       </geometry>
         <origin xyz = "-0.047 -0.013 0.044 " rpy = " 1.5708 0 1.5708"/>
@@ -156,5 +191,6 @@
     <collision>
       <geometry>
-       <mesh filename="package://pro450_description/meshes/pro_gripper_left2.dae"/>
+       <mesh filename="package://pro450_description/meshes/pro_gripper_left2.dae"
+             scale="$(arg collision_mesh_scale) $(arg collision_mesh_scale) $(arg collision_mesh_scale)"/>
       </geometry>
         <origin xyz = "-0.0 0.03 0.004 " rpy = " 3.14159 0 1.5708"/>
@@ -170,5 +206,6 @@
     <collision>
       <geometry>
-       <mesh filename="package://pro450_description/meshes/pro_gripper_left3.dae"/>
+       <mesh filename="package://pro450_description/meshes/pro_gripper_left3.dae"
+             scale="$(arg collision_mesh_scale) $(arg collision_mesh_scale) $(arg collision_mesh_scale)"/>
       </geometry>
     <origin xyz = "0 -0.03 0.012 " rpy = " 1.5708 3.14159 1.5708"/>
@@ -184,5 +221,6 @@
     <collision>
       <geometry>
-       <mesh filename="package://pro450_description/meshes/pro_gripper_right1.dae"/>
+       <mesh filename="package://pro450_description/meshes/pro_gripper_right1.dae"
+             scale="$(arg collision_mesh_scale) $(arg collision_mesh_scale) $(arg collision_mesh_scale)"/>
       </geometry>
         <origin xyz = "0.047 -0.013 -0.046 " rpy = " 1.5708 3.14 -1.5708"/>
@@ -198,5 +236,6 @@
     <collision>
       <geometry>
-       <mesh filename="package://pro450_description/meshes/pro_gripper_right2.dae"/>
+       <mesh filename="package://pro450_description/meshes/pro_gripper_right2.dae"
+             scale="$(arg collision_mesh_scale) $(arg collision_mesh_scale) $(arg collision_mesh_scale)"/>
       </geometry>
         <origin xyz = "0 0.03 -0.005 " rpy = " 0 0 1.5708"/>
@@ -212,5 +251,6 @@
     <collision>
       <geometry>
-       <mesh filename="package://pro450_description/meshes/pro_gripper_right3.dae"/>
+       <mesh filename="package://pro450_description/meshes/pro_gripper_right3.dae"
+             scale="$(arg collision_mesh_scale) $(arg collision_mesh_scale) $(arg collision_mesh_scale)"/>
       </geometry>
     <origin xyz = "-0.014 -0.029 0.004 " rpy = " 3.14 0 -1.5708"/>
@@ -219,5 +259,5 @@
   <joint name="joint1" type="revolute">
     <axis xyz="0 0 1"/>
-    <limit effort = "1000.0" lower = "-2.8274" upper = "2.8274" velocity = "0"/>
+    <limit effort = "1000.0" lower = "-2.8274" upper = "2.8274" velocity = "1.5"/>
     <parent link="base"/>
     <child link="link1"/>
@@ -226,5 +266,5 @@
   <joint name="joint2" type="revolute">
     <axis xyz="1 0 0"/>
-    <limit effort = "1000.0" lower = "-2.1816" upper = "2.1816" velocity = "0"/>
+    <limit effort = "1000.0" lower = "-2.1816" upper = "2.1816" velocity = "1.5"/>
     <parent link="link1"/>
     <child link="link2"/>
@@ -233,5 +273,5 @@
   <joint name="joint3" type="revolute">
     <axis xyz=" 1 0 0"/>
-    <limit effort = "1000.0" lower = "-2.6878" upper = "2.6878" velocity = "0"/>
+    <limit effort = "1000.0" lower = "-2.6878" upper = "2.6878" velocity = "1.5"/>
     <parent link="link2"/>
     <child link="link3"/>
@@ -240,5 +280,5 @@
   <joint name="joint4" type="revolute">
     <axis xyz=" 1 0 0"/>
-    <limit effort = "1000.0" lower = "-2.8274" upper = "2.8274" velocity = "0"/>
+    <limit effort = "1000.0" lower = "-2.8274" upper = "2.8274" velocity = "1.5"/>
     <parent link="link3"/>
     <child link="link4"/>
@@ -247,5 +287,5 @@
   <joint name="joint5" type="revolute">
     <axis xyz="0 0 1"/>
-    <limit effort = "1000.0" lower = "-2.8274" upper = "2.8274" velocity = "0"/>
+    <limit effort = "1000.0" lower = "-2.8274" upper = "2.8274" velocity = "1.5"/>
     <parent link="link4"/>
     <child link="link5"/>
@@ -254,5 +294,5 @@
   <joint name="joint6" type="revolute">
     <axis xyz="1 0 0"/>
-    <limit effort = "1000.0" lower = "-2.8797" upper = "2.8797" velocity = "0"/>
+    <limit effort = "1000.0" lower = "-2.8797" upper = "2.8797" velocity = "1.5"/>
     <parent link="link5"/>
     <child link="link6"/>
@@ -271,5 +311,8 @@
   <joint name="gripper_controller" type="revolute">
     <axis xyz="0 0 1"/>
-    <limit effort = "1000.0" lower = "0" upper = "1" velocity = "0"/>
+    <!-- Gazebo can settle a few microradians below the nominal open value.
+         Keep a narrow numerical margin while preserving the physical 0..1
+         command range used by the F100 controller. -->
+    <limit effort = "1000.0" lower = "-0.01" upper = "1" velocity = "1.5"/>
     <parent link="gripper_base"/>
     <child link="gripper_left3"/>
@@ -278,5 +321,5 @@
   <joint name="gripper_base_to_gripper_left2" type="revolute">
     <axis xyz="0 0 1"/>
-    <limit effort = "1000.0" lower = "-0.8" upper = "0.5" velocity = "0"/>
+    <limit effort = "1000.0" lower = "-1" upper = "1" velocity = "1.5"/>
     <parent link="gripper_base"/>
     <child link="gripper_left2"/>
@@ -286,5 +329,5 @@
   <joint name="gripper_left3_to_gripper_left1" type="revolute">
     <axis xyz="0 0 1"/>
-    <limit effort = "1000.0" lower = "-0.5" upper = "0.5" velocity = "0"/>
+    <limit effort = "1000.0" lower = "-1" upper = "1" velocity = "1.5"/>
     <parent link="gripper_left3"/>
     <child link="gripper_left1"/>
@@ -294,5 +337,5 @@
   <joint name="gripper_base_to_gripper_right3" type="revolute">
     <axis xyz="0 0 1"/>
-    <limit effort = "1000.0" lower = "1" upper = "0" velocity = "0"/>
+    <limit effort = "1000.0" lower = "-1" upper = "1" velocity = "1.5"/>
     <parent link="gripper_base"/>
     <child link="gripper_right3"/>
@@ -302,5 +345,5 @@
   <joint name="gripper_base_to_gripper_right2" type="revolute">
     <axis xyz="0 0 1"/>
-    <limit effort = "1000.0" lower = "-0.5" upper = "0.8" velocity = "0"/>
+    <limit effort = "1000.0" lower = "-1" upper = "1" velocity = "1.5"/>
     <parent link="gripper_base"/>
     <child link="gripper_right2"/>
@@ -310,5 +353,5 @@
   <joint name="gripper_right3_to_gripper_right1" type="revolute">
     <axis xyz="0 0 1"/>
-    <limit effort = "1000.0" lower = "-0.5" upper = "0.5" velocity = "0"/>
+    <limit effort = "1000.0" lower = "-1" upper = "1" velocity = "1.5"/>
     <parent link="gripper_right3"/>
     <child link="gripper_right1"/>
@@ -316,14 +359,34 @@
     <mimic joint="gripper_controller" multiplier="1.0" offset="0" />
   </joint>
-  <!-- Keep the exact eye-in-hand D435 mounting convention used by TM5/RG2. -->
+  <!-- Final F100 underside mounting datum, established from the two verified
+       points BASE-2=(0.023016, 0.038663, -0.033656) m and
+       BASE-4=(-0.024984, 0.038663, -0.033656) m in gripper_base.  Their
+       separation is 48 mm and their midpoint is the bracket datum.  Because
+       the preserved D435 orientation makes the vendor mesh grow 25 mm into
+       the gripper from camera_bottom_screw_frame, translate the complete
+       camera one housing height downward so its upper face meets that datum. -->
+  <xacro:property name="d435_mount_x" value="-0.000984"/>
+  <xacro:property name="d435_mount_y" value="0.038663"/>
+  <xacro:property name="d435_mount_z" value="-0.058656"/>
+  <!-- Keep the already-validated D435 body orientation unchanged. -->
+  <xacro:property name="d435_mount_yaw" value="1.5707963267948966"/>
   <link name="tmvision_camera_frame"/>
   <joint name="tmvision_camera_joint" type="fixed">
-    <parent link="link6"/>
+    <parent link="gripper_base"/>
     <child link="tmvision_camera_frame"/>
-    <origin xyz="0.0175 0.1243 0.01933" rpy="0 -1.5707 -1.5707"/>
-  </joint>
-  <xacro:sensor_d435 parent="link6" name="camera"
+    <origin xyz="${d435_mount_x} ${d435_mount_y} ${d435_mount_z}"
+            rpy="0 0 ${d435_mount_yaw}"/>
+  </joint>
+  <xacro:sensor_d435 parent="gripper_base" name="camera"
                      use_nominal_extrinsics="true" add_plug="false" use_mesh="true">
-    <origin xyz="0.0 0.1243 0.02373" rpy="1.5708 -1.5708 0.0"/>
+    <origin xyz="${d435_mount_x} ${d435_mount_y} ${d435_mount_z}"
+            rpy="0 0 ${d435_mount_yaw}"/>
   </xacro:sensor_d435>
+  <!-- Preserve the D435 mounting link through URDF-to-SDF conversion, then
+       attach the Fortress RGB-D sensor to that same physical mounting link. -->
+  <gazebo reference="camera_joint"><preserveFixedJoint>true</preserveFixedJoint></gazebo>
+  <xacro:pro450_d435_gz_rgbd_camera parent_link="camera_bottom_screw_frame"/>
+  <xacro:if value="$(arg use_gz_control)">
+    <xacro:pro450_gz_ros2_control/>
+  </xacro:if>
 </robot>
