Commit message: chore: update code structure and remove redundant changes

File: agbot/pro450_description/urdf/pro450_f100.urdf.xacro (robot description, xacro)
@@ -2,391 +2,7 @@
 <robot xmlns:xacro="http://www.ros.org/wiki/xacro" name="mycobot_pro_450_f100">
   <xacro:arg name="use_gz_control" default="false"/>
+  <xacro:arg name="use_fake_hardware" default="false"/>
   <xacro:arg name="collision_mesh_scale" default="1.0"/>
-  <!-- Vendor geometry and kinematic chain imported from Elephant Robotics
-       mycobot_ros2 Humble commit 3999e2c.  The D435 transform deliberately
-       matches the existing TM5 leaf-simulation description. -->
-  <xacro:include filename="$(find realsense2_description)/urdf/_d435.urdf.xacro"/>
-  <xacro:include filename="$(find pro450_description)/urdf/pro450_gz_plugins.xacro"/>
-<xacro:property name="width" value=".2" />
-  <!-- Keep the same floor installation datum as the previous TM5 environment. -->
-  <xacro:property name="mount_plate_height" value="0.05"/>
-  <link name="base_root"/>
-  <link name="mount_plate_link">
-    <visual>
-      <origin xyz="0 0 ${mount_plate_height / 2.0}" rpy="0 0 0"/>
-      <geometry><box size="0.50 0.50 ${mount_plate_height}"/></geometry>
-      <material name="mount_plate_gray"><color rgba="0.55 0.55 0.58 1.0"/></material>
-    </visual>
-    <collision>
-      <origin xyz="0 0 ${mount_plate_height / 2.0}" rpy="0 0 0"/>
-      <geometry><box size="0.50 0.50 ${mount_plate_height}"/></geometry>
-    </collision>
-    <inertial><mass value="5.0"/><inertia ixx="0.1" ixy="0" ixz="0" iyy="0.1" iyz="0" izz="0.1"/></inertial>
-  </link>
-  <joint name="root_to_plate" type="fixed">
-    <parent link="base_root"/><child link="mount_plate_link"/><origin xyz="0 0 0" rpy="0 0 0"/>
-  </joint>
-  <link name="base">
-    <visual>
-      <geometry>
-       <mesh filename="package://pro450_description/meshes/PRO450_J1.dae"/>
-      </geometry>
-      <origin xyz = "-0.108 -0.003 0 " rpy = " 0 0 -1.5708"/>
-    </visual>
-    <collision>
-      <geometry>
-       <mesh filename="package://pro450_description/meshes/PRO450_J1.dae"
-             scale="$(arg collision_mesh_scale) $(arg collision_mesh_scale) $(arg collision_mesh_scale)"/>
-        </geometry>
-        <origin xyz = "-0.108 -0.003 0 " rpy = " 0 0 -1.5708"/>
-    </collision>
-  </link>
-  <link name="link1">
-    <visual>
-      <geometry>
-       <mesh filename="package://pro450_description/meshes/PRO450_J2.dae"/>
-      </geometry>
-      <origin xyz = "0.0015 -0.0392 0.0 " rpy = " -1.5708 0 -3.14159 "/>
-    </visual>
-    <collision>
-     <geometry>
-       <mesh filename="package://pro450_description/meshes/PRO450_J2.dae"
-             scale="$(arg collision_mesh_scale) $(arg collision_mesh_scale) $(arg collision_mesh_scale)"/>
-      </geometry>
-      <origin xyz = "0.0015 -0.0392 0.0 " rpy = " -1.5708 0 -3.14159 "/>
-    </collision>
-  </link>
-  <joint name="plate_to_arm_base" type="fixed">
-    <parent link="mount_plate_link"/><child link="base"/>
-    <origin xyz="0 0 ${mount_plate_height}" rpy="0 0 0"/>
-  </joint>
-  <link name="link2">
-    <visual>
-      <geometry>
-       <mesh filename="package://pro450_description/meshes/PRO450_J3.dae"/>
-      </geometry>
-    <origin xyz = "0.0598 0.005 -0.203 " rpy = " 0 0 1.5708 "/>
-    </visual>
-    <collision>
-      <geometry>
-       <mesh filename="package://pro450_description/meshes/PRO450_J3.dae"
-             scale="$(arg collision_mesh_scale) $(arg collision_mesh_scale) $(arg collision_mesh_scale)"/>
-      </geometry>
-      <origin xyz = "0.0598  0.005 -0.203 " rpy = " 0 0 1.5708"/>
-    </collision>
-  </link>
-  <link name="link3">
-    <visual>
-      <geometry>
-       <mesh filename="package://pro450_description/meshes/PRO450_J4.dae"/>
-      </geometry>
-      <origin xyz = "0.07 0.005 -0.383 " rpy = " 0 0 1.5708"/>
-    </visual>
-    <collision>
-      <geometry>
-       <mesh filename="package://pro450_description/meshes/PRO450_J4.dae"
-             scale="$(arg collision_mesh_scale) $(arg collision_mesh_scale) $(arg collision_mesh_scale)"/>
-      </geometry>
-      <origin xyz = "0.07 0.005 -0.383" rpy = " 0 0 1.5708"/>
-    </collision>
-  </link>
-  <link name="link4">
-    <visual>
-      <geometry>
-       <mesh filename="package://pro450_description/meshes/PRO450_J5.dae"/>
-      </geometry>
-    <origin xyz = "-0.014 0 0.0 " rpy = " 0 -1.5708 0"/>
-    </visual>
-    <collision>
-       <geometry>
-       <mesh filename="package://pro450_description/meshes/PRO450_J5.dae"
-             scale="$(arg collision_mesh_scale) $(arg collision_mesh_scale) $(arg collision_mesh_scale)"/>
-      </geometry>
-      <origin xyz = "-0.014 0 0.0 " rpy = " 0 -1.5708 0"/>
-    </collision>
-  </link>
-  <link name="link5">
-    <visual>
-      <geometry>
-       <mesh filename="package://pro450_description/meshes/PRO450_J6.dae"/>
-      </geometry>
-    <origin xyz = "0.004 -0.024 -0.655 " rpy = " 0 0 0"/>
-    </visual>
-    <collision>
-      <geometry>
-       <mesh filename="package://pro450_description/meshes/PRO450_J6.dae"
-             scale="$(arg collision_mesh_scale) $(arg collision_mesh_scale) $(arg collision_mesh_scale)"/>
-      </geometry>
-    <origin xyz = "0.004 -0.024 -0.655 " rpy = " 0 0 0"/>
-    </collision>
-  </link>
-  <link name="link6">
-    <visual>
-      <geometry>
-       <mesh filename="package://pro450_description/meshes/PRO450_J6_end.dae"/>
-      </geometry>
-    <origin xyz = "0 0 0 " rpy = " 3.14159 0 0"/>
-    </visual>
-    <collision>
-      <geometry>
-       <mesh filename="package://pro450_description/meshes/PRO450_J6_end.dae"
-             scale="$(arg collision_mesh_scale) $(arg collision_mesh_scale) $(arg collision_mesh_scale)"/>
-      </geometry>
-    <origin xyz = "0 0 0 " rpy = " 3.14159 0 0"/>
-    </collision>
-  </link>
-  <link name="gripper_connection">
-    <visual>
-      <geometry>
-       <mesh filename="package://pro450_description/meshes/mygripper_f100_connection.dae"/>
-      </geometry>
-    <origin xyz = "-0.03 0.014 0 " rpy = " 0  0 -1.5708"/>
-    </visual>
-    <collision>
-      <geometry>
-       <mesh filename="package://pro450_description/meshes/mygripper_f100_connection.dae"
-             scale="$(arg collision_mesh_scale) $(arg collision_mesh_scale) $(arg collision_mesh_scale)"/>
-      </geometry>
-    <origin xyz = "-0.03 0.014 0 " rpy = " 0  0 -1.5708"/>
-    </collision>
-  </link>
-  <link name="gripper_base">
-    <visual>
-      <geometry>
-       <mesh filename="package://pro450_description/meshes/pro_gripper_base.dae"/>
-      </geometry>
-    <origin xyz = "-0.107 0.012 0.0 " rpy = " 1.5708  0 1.5708"/>
-    </visual>
-    <collision>
-      <geometry>
-       <mesh filename="package://pro450_description/meshes/pro_gripper_base.dae"
-             scale="$(arg collision_mesh_scale) $(arg collision_mesh_scale) $(arg collision_mesh_scale)"/>
-      </geometry>
-    <origin xyz = "-0.107 0.012 0.0 " rpy = " 1.5708  0 1.5708"/>
-    </collision>
-  </link>
-  <link name="gripper_left1">
-    <visual>
-      <geometry>
-       <!--- 0.0 0 -0.04 -->
-       <mesh filename="package://pro450_description/meshes/pro_gripper_left1.dae"/>
-      </geometry>
-    <origin xyz = "-0.047 -0.013 0.044 " rpy = " 1.5708 0 1.5708"/>
-    </visual>
-    <collision>
-      <geometry>
-       <mesh filename="package://pro450_description/meshes/pro_gripper_left1.dae"
-             scale="$(arg collision_mesh_scale) $(arg collision_mesh_scale) $(arg collision_mesh_scale)"/>
-      </geometry>
-        <origin xyz = "-0.047 -0.013 0.044 " rpy = " 1.5708 0 1.5708"/>
-    </collision>
-  </link>
-  <link name="gripper_left2">
-    <visual>
-      <geometry>
-       <mesh filename="package://pro450_description/meshes/pro_gripper_left2.dae"/>
-      </geometry>
-    <origin xyz = "-0.0 0.03 0.004 " rpy = " 3.14159 0 1.5708"/>
-    </visual>
-    <collision>
-      <geometry>
-       <mesh filename="package://pro450_description/meshes/pro_gripper_left2.dae"
-             scale="$(arg collision_mesh_scale) $(arg collision_mesh_scale) $(arg collision_mesh_scale)"/>
-      </geometry>
-        <origin xyz = "-0.0 0.03 0.004 " rpy = " 3.14159 0 1.5708"/>
-    </collision>
-  </link>
-  <link name="gripper_left3">
-    <visual>
-      <geometry>
-       <mesh filename="package://pro450_description/meshes/pro_gripper_left3.dae"/>
-      </geometry>
-    <origin xyz = "0 -0.03 0.012 " rpy = " 1.5708 3.14159 1.5708"/>
-    </visual>
-    <collision>
-      <geometry>
-       <mesh filename="package://pro450_description/meshes/pro_gripper_left3.dae"
-             scale="$(arg collision_mesh_scale) $(arg collision_mesh_scale) $(arg collision_mesh_scale)"/>
-      </geometry>
-    <origin xyz = "0 -0.03 0.012 " rpy = " 1.5708 3.14159 1.5708"/>
-    </collision>
-  </link>
-  <link name="gripper_right1">
-    <visual>
-      <geometry>
-       <mesh filename="package://pro450_description/meshes/pro_gripper_right1.dae"/>
-      </geometry>
-    <origin xyz = "0.047 -0.013 -0.046 " rpy = " 1.5708 3.14 -1.5708"/>
-    </visual>
-    <collision>
-      <geometry>
-       <mesh filename="package://pro450_description/meshes/pro_gripper_right1.dae"
-             scale="$(arg collision_mesh_scale) $(arg collision_mesh_scale) $(arg collision_mesh_scale)"/>
-      </geometry>
-        <origin xyz = "0.047 -0.013 -0.046 " rpy = " 1.5708 3.14 -1.5708"/>
-    </collision>
-  </link>
-  <link name="gripper_right2">
-    <visual>
-      <geometry>
-       <mesh filename="package://pro450_description/meshes/pro_gripper_right2.dae"/>
-      </geometry>
-    <origin xyz = "0 0.03 -0.005 " rpy = " 0 0 1.5708"/>
-    </visual>
-    <collision>
-      <geometry>
-       <mesh filename="package://pro450_description/meshes/pro_gripper_right2.dae"
-             scale="$(arg collision_mesh_scale) $(arg collision_mesh_scale) $(arg collision_mesh_scale)"/>
-      </geometry>
-        <origin xyz = "0 0.03 -0.005 " rpy = " 0 0 1.5708"/>
-    </collision>
-  </link>
-  <link name="gripper_right3">
-    <visual>
-      <geometry>
-       <mesh filename="package://pro450_description/meshes/pro_gripper_right3.dae"/>
-      </geometry>
-    <origin xyz = "-0.014 -0.029 0.004 " rpy = " 3.14 0 -1.5708"/>
-    </visual>
-    <collision>
-      <geometry>
-       <mesh filename="package://pro450_description/meshes/pro_gripper_right3.dae"
-             scale="$(arg collision_mesh_scale) $(arg collision_mesh_scale) $(arg collision_mesh_scale)"/>
-      </geometry>
-    <origin xyz = "-0.014 -0.029 0.004 " rpy = " 3.14 0 -1.5708"/>
-    </collision>
-  </link>
-  <joint name="joint1" type="revolute">
-    <axis xyz="0 0 1"/>
-    <limit effort = "1000.0" lower = "-2.8274" upper = "2.8274" velocity = "1.5"/>
-    <parent link="base"/>
-    <child link="link1"/>
-    <origin xyz= "0 0 0.210" rpy = "0 0 0"/>
-  </joint>
-  <joint name="joint2" type="revolute">
-    <axis xyz="1 0 0"/>
-    <limit effort = "1000.0" lower = "-2.1816" upper = "2.1816" velocity = "1.5"/>
-    <parent link="link1"/>
-    <child link="link2"/>
-    <origin xyz= "0.0 -0.048 0" rpy = "0 0 -1.5708"/>
-  </joint>
-  <joint name="joint3" type="revolute">
-    <axis xyz=" 1 0 0"/>
-    <limit effort = "1000.0" lower = "-2.6878" upper = "2.6878" velocity = "1.5"/>
-    <parent link="link2"/>
-    <child link="link3"/>
-    <origin xyz= "-0.01 0 0.18  " rpy = "0 0 0"/>
-  </joint>
-  <joint name="joint4" type="revolute">
-    <axis xyz=" 1 0 0"/>
-    <limit effort = "1000.0" lower = "-2.8274" upper = "2.8274" velocity = "1.5"/>
-    <parent link="link3"/>
-    <child link="link4"/>
-    <origin xyz= "0 0 0.173" rpy = "0 0 0"/>
-  </joint>
-  <joint name="joint5" type="revolute">
-    <axis xyz="0 0 1"/>
-    <limit effort = "1000.0" lower = "-2.8274" upper = "2.8274" velocity = "1.5"/>
-    <parent link="link4"/>
-    <child link="link5"/>
-    <origin xyz= "0.0455 0 0.097" rpy = "0 0 0"/>
-  </joint>
-  <joint name="joint6" type="revolute">
-    <axis xyz="1 0 0"/>
-    <limit effort = "1000.0" lower = "-2.8797" upper = "2.8797" velocity = "1.5"/>
-    <parent link="link5"/>
-    <child link="link6"/>
-    <origin xyz= "0 0.04 0" rpy = "0 0 1.5708"/>
-  </joint>
-  <joint name="joint6_to_gripper_connect" type="fixed">
-    <parent link="link6"/>
-    <child link="gripper_connection"/>
-     <origin xyz= "0.03 0.0 -0.01" rpy = "-1.5708 0 -1.5708"/>
-  </joint>
-  <joint name="joint6_to_gripper_base" type="fixed">
-    <parent link="gripper_connection"/>
-    <child link="gripper_base"/>
-     <origin xyz= "0 -0.02 0.0364" rpy = "1.5708 0 0"/>
-  </joint>
-  <joint name="gripper_controller" type="revolute">
-    <axis xyz="0 0 1"/>
-    <!-- Gazebo can settle a few microradians below the nominal open value.
-         Keep a narrow numerical margin while preserving the physical 0..1
-         command range used by the F100 controller. -->
-    <limit effort = "1000.0" lower = "-0.01" upper = "1" velocity = "1.5"/>
-    <parent link="gripper_base"/>
-    <child link="gripper_left3"/>
-    <origin xyz= "-0.018 0.016 -0.02" rpy = "0 0 0"/>
-  </joint>
-  <joint name="gripper_base_to_gripper_left2" type="revolute">
-    <axis xyz="0 0 1"/>
-    <limit effort = "1000.0" lower = "-1" upper = "1" velocity = "1.5"/>
-    <parent link="gripper_base"/>
-    <child link="gripper_left2"/>
-    <origin xyz= "-0.0445 -0.004 -0.02" rpy = "0 0 0"/>
-    <mimic joint="gripper_controller" multiplier="1.0" offset="0" />
-  </joint>
-  <joint name="gripper_left3_to_gripper_left1" type="revolute">
-    <axis xyz="0 0 1"/>
-    <limit effort = "1000.0" lower = "-1" upper = "1" velocity = "1.5"/>
-    <parent link="gripper_left3"/>
-    <child link="gripper_left1"/>
-    <origin xyz= "0.01 0.06 0.0" rpy = "0 0 0"/>
-    <mimic joint="gripper_controller" multiplier="-1.0" offset="0" />
-  </joint>
-  <joint name="gripper_base_to_gripper_right3" type="revolute">
-    <axis xyz="0 0 1"/>
-    <limit effort = "1000.0" lower = "-1" upper = "1" velocity = "1.5"/>
-    <parent link="gripper_base"/>
-    <child link="gripper_right3"/>
-    <origin xyz= "0.018 0.015 -0.0212" rpy = "0 0 0"/>
-    <mimic joint="gripper_controller" multiplier="-1.0" offset="0" />
-  </joint>
-  <joint name="gripper_base_to_gripper_right2" type="revolute">
-    <axis xyz="0 0 1"/>
-    <limit effort = "1000.0" lower = "-1" upper = "1" velocity = "1.5"/>
-    <parent link="gripper_base"/>
-    <child link="gripper_right2"/>
-    <origin xyz= "0.0442 -0.004 -0.02" rpy = "0 0 0"/>
-    <mimic joint="gripper_controller" multiplier="-1.0" offset="0" />
-  </joint>
-  <joint name="gripper_right3_to_gripper_right1" type="revolute">
-    <axis xyz="0 0 1"/>
-    <limit effort = "1000.0" lower = "-1" upper = "1" velocity = "1.5"/>
-    <parent link="gripper_right3"/>
-    <child link="gripper_right1"/>
-    <origin xyz= "-0.01 0.061 0.001" rpy = "0 0 0"/>
-    <mimic joint="gripper_controller" multiplier="1.0" offset="0" />
-  </joint>
-  <!-- Final F100 underside mounting datum, established from the two verified
-       points BASE-2=(0.023016, 0.038663, -0.033656) m and
-       BASE-4=(-0.024984, 0.038663, -0.033656) m in gripper_base.  Their
-       separation is 48 mm and their midpoint is the bracket datum.  Because
-       the preserved D435 orientation makes the vendor mesh grow 25 mm into
-       the gripper from camera_bottom_screw_frame, translate the complete
-       camera one housing height downward so its upper face meets that datum. -->
-  <xacro:property name="d435_mount_x" value="-0.000984"/>
-  <xacro:property name="d435_mount_y" value="0.038663"/>
-  <xacro:property name="d435_mount_z" value="-0.058656"/>
-  <!-- Keep the already-validated D435 body orientation unchanged. -->
-  <xacro:property name="d435_mount_yaw" value="1.5707963267948966"/>
-  <link name="tmvision_camera_frame"/>
-  <joint name="tmvision_camera_joint" type="fixed">
-    <parent link="gripper_base"/>
-    <child link="tmvision_camera_frame"/>
-    <origin xyz="${d435_mount_x} ${d435_mount_y} ${d435_mount_z}"
-            rpy="0 0 ${d435_mount_yaw}"/>
-  </joint>
-  <xacro:sensor_d435 parent="gripper_base" name="camera"
-                     use_nominal_extrinsics="true" add_plug="false" use_mesh="true">
-    <origin xyz="${d435_mount_x} ${d435_mount_y} ${d435_mount_z}"
-            rpy="0 0 ${d435_mount_yaw}"/>
-  </xacro:sensor_d435>
-  <!-- Preserve the D435 mounting link through URDF-to-SDF conversion, then
-       attach the Fortress RGB-D sensor to that same physical mounting link. -->
-  <gazebo reference="camera_joint"><preserveFixedJoint>true</preserveFixedJoint></gazebo>
-  <xacro:pro450_d435_gz_rgbd_camera parent_link="camera_bottom_screw_frame"/>
-  <xacro:if value="$(arg use_gz_control)">
-    <xacro:pro450_gz_ros2_control/>
-  </xacro:if>
+  <xacro:arg name="use_floor_mount" default="true"/>
+  <xacro:include filename="$(find pro450_description)/urdf/pro450_f100_body.xacro"/>
 </robot>

File: agbot/pro450_description/urdf/pro450_gz_plugins.xacro (robot description, xacro)
@@ -3,5 +3,5 @@
   <!-- Fortress-native RGB-D sensor.  The launch bridge maps /camera_gz to
        the same ROS image, depth, and point-cloud topics as the TM5 scene. -->
-  <xacro:macro name="pro450_d435_gz_rgbd_camera" params="parent_link:='camera_bottom_screw_frame'">
+  <xacro:macro name="pro450_d435_gz_rgbd_camera" params="parent_link:='camera_depth_frame'">
     <gazebo reference="${parent_link}">
       <sensor name="d435_depth_camera" type="rgbd_camera">
@@ -22,4 +22,35 @@
     </gazebo>
   </xacro:macro>
+  <!-- Chassis Orbbec stand-in for mobile SLAM (longer range for corridors).
+       Fortress rgbd_camera looks along +X of parent.  Parent is
+       camera_depth_frame (X-forward).  Stamp as camera_depth_optical_frame
+       so depthimage_to_laserscan / RTAB-Map use ROS optical (Z-forward);
+       URDF optical joint maps optical Z → robot forward. -->
+  <xacro:macro name="pro450_chassis_gz_rgbd_camera" params="parent_link:='camera_depth_frame' far:='8.0'">
+    <gazebo reference="${parent_link}">
+      <sensor name="chassis_rgbd_camera" type="rgbd_camera">
+        <pose>0 0 0 0 0 0</pose>
+        <gz_frame_id>camera_depth_optical_frame</gz_frame_id>
+        <always_on>true</always_on>
+        <update_rate>15.0</update_rate>
+        <visualize>true</visualize>
+        <topic>/camera_gz</topic>
+        <camera>
+          <horizontal_fov>1.396</horizontal_fov>
+          <image><width>640</width><height>480</height><format>R8G8B8</format></image>
+          <clip><near>0.15</near><far>${far}</far></clip>
+        </camera>
+      </sensor>
+    </gazebo>
+  </xacro:macro>
+  <xacro:macro name="pro450_arm_joint_interfaces">
+    <joint name="joint1"><command_interface name="position"/><state_interface name="position"/><state_interface name="velocity"/></joint>
+    <joint name="joint2"><command_interface name="position"/><state_interface name="position"/><state_interface name="velocity"/></joint>
+    <joint name="joint3"><command_interface name="position"/><state_interface name="position"/><state_interface name="velocity"/></joint>
+    <joint name="joint4"><command_interface name="position"/><state_interface name="position"/><state_interface name="velocity"/></joint>
+    <joint name="joint5"><command_interface name="position"/><state_interface name="position"/><state_interface name="velocity"/></joint>
+    <joint name="joint6"><command_interface name="position"/><state_interface name="position"/><state_interface name="velocity"/></joint>
+    <joint name="gripper_controller"><command_interface name="position"/><state_interface name="position"/><state_interface name="velocity"/></joint>
+  </xacro:macro>
   <xacro:macro name="pro450_gz_ros2_control">
     <ros2_control name="Pro450GazeboSystem" type="system">
@@ -27,11 +58,5 @@
         <plugin>gz_ros2_control/GazeboSimSystem</plugin>
       </hardware>
-      <joint name="joint1"><command_interface name="position"/><state_interface name="position"/><state_interface name="velocity"/></joint>
-      <joint name="joint2"><command_interface name="position"/><state_interface name="position"/><state_interface name="velocity"/></joint>
-      <joint name="joint3"><command_interface name="position"/><state_interface name="position"/><state_interface name="velocity"/></joint>
-      <joint name="joint4"><command_interface name="position"/><state_interface name="position"/><state_interface name="velocity"/></joint>
-      <joint name="joint5"><command_interface name="position"/><state_interface name="position"/><state_interface name="velocity"/></joint>
-      <joint name="joint6"><command_interface name="position"/><state_interface name="position"/><state_interface name="velocity"/></joint>
-      <joint name="gripper_controller"><command_interface name="position"/><state_interface name="position"/><state_interface name="velocity"/></joint>
+      <xacro:pro450_arm_joint_interfaces/>
     </ros2_control>
     <gazebo reference="base_root"><kinematic>true</kinematic></gazebo>
@@ -45,3 +70,17 @@
     </gazebo>
   </xacro:macro>
+  <!-- Offline / RViz control without Gazebo: mock hardware for arm + myAGV wheels. -->
+  <xacro:macro name="pro450_myagv_fake_ros2_control">
+    <ros2_control name="Pro450MyAgvFakeSystem" type="system">
+      <hardware>
+        <plugin>mock_components/GenericSystem</plugin>
+        <param name="calculate_dynamics">false</param>
+      </hardware>
+      <xacro:pro450_arm_joint_interfaces/>
+      <joint name="right_rear_wheel_joint"><command_interface name="position"/><state_interface name="position"/><state_interface name="velocity"/></joint>
+      <joint name="right_front_wheel_joint"><command_interface name="position"/><state_interface name="position"/><state_interface name="velocity"/></joint>
+      <joint name="left_front_wheel_joint"><command_interface name="position"/><state_interface name="position"/><state_interface name="velocity"/></joint>
+      <joint name="left_rear_wheel_joint"><command_interface name="position"/><state_interface name="position"/><state_interface name="velocity"/></joint>
+    </ros2_control>
+  </xacro:macro>
 </robot>
