Commit message: feat: Add leaf inspection and wheel joint state publishing scripts
- Introduced `pro450_myagv_leaf_environment.sh` to set up the Gazebo and Nav2 environment for plant inspections.
- Created `pro450_myagv_leaf_inspection.py` for executing leaf pinch inspections on specified plants.
- Added `pro450_myagv_leaf_inspection.sh` for interactive selection of plants for inspection.
- Implemented `pro450_myagv_wheel_joint_states.py` to publish wheel joint states for the robot_state_publisher.
- Added a compiled Python file for wheel joint states to improve performance.

File: agbot/pro450_description/urdf/pro450_f100_body.xacro (robot description, xacro)
@@ -401,8 +401,16 @@
          (10.6, 17.5, 12.5) mm away from camera_bottom_screw_frame. -->
     <gazebo reference="camera_joint"><preserveFixedJoint>true</preserveFixedJoint></gazebo>
-    <xacro:pro450_d435_gz_rgbd_camera parent_link="camera_depth_frame"/>
+    <xacro:pro450_d435_gz_rgbd_camera
+      parent_link="camera_depth_frame"
+      topic="/wrist_camera_gz"
+      frame_id="camera_depth_optical_frame"/>
   </xacro:if>
   <xacro:if value="$(arg use_gz_control)">
-    <xacro:pro450_gz_ros2_control/>
+    <xacro:if value="$(arg use_floor_mount)">
+      <xacro:pro450_gz_ros2_control root_link="base_root" root_kinematic="true"/>
+    </xacro:if>
+    <xacro:unless value="$(arg use_floor_mount)">
+      <xacro:pro450_gz_ros2_control root_link="base_footprint" root_kinematic="false"/>
+    </xacro:unless>
   </xacro:if>
   <xacro:if value="$(arg use_fake_hardware)">

File: agbot/pro450_description/urdf/pro450_gz_plugins.xacro (robot description, xacro)
@@ -3,5 +3,6 @@
   <!-- Fortress-native RGB-D sensor.  The launch bridge maps /camera_gz to
        the same ROS image, depth, and point-cloud topics as the TM5 scene. -->
-  <xacro:macro name="pro450_d435_gz_rgbd_camera" params="parent_link:='camera_depth_frame'">
+  <xacro:macro name="pro450_d435_gz_rgbd_camera"
+               params="parent_link:='camera_depth_frame' topic:='/camera_gz' frame_id:='camera_depth_optical_frame'">
     <gazebo reference="${parent_link}">
       <sensor name="d435_depth_camera" type="rgbd_camera">
@@ -9,9 +10,9 @@
              sensor must use its unflipped local gaze to face the plant. -->
         <pose>0 0 0 0 0 0</pose>
-        <gz_frame_id>camera_depth_optical_frame</gz_frame_id>
+        <gz_frame_id>${frame_id}</gz_frame_id>
         <always_on>true</always_on>
         <update_rate>10.0</update_rate>
         <visualize>false</visualize>
-        <topic>/camera_gz</topic>
+        <topic>${topic}</topic>
         <camera>
           <horizontal_fov>1.047</horizontal_fov>
@@ -27,13 +28,14 @@
        so depthimage_to_laserscan / RTAB-Map use ROS optical (Z-forward);
        URDF optical joint maps optical Z → robot forward. -->
-  <xacro:macro name="pro450_chassis_gz_rgbd_camera" params="parent_link:='camera_depth_frame' far:='8.0'">
+  <xacro:macro name="pro450_chassis_gz_rgbd_camera"
+               params="parent_link:='nav_camera_depth_frame' far:='8.0' topic:='/nav_camera_gz' frame_id:='nav_camera_depth_optical_frame'">
     <gazebo reference="${parent_link}">
       <sensor name="chassis_rgbd_camera" type="rgbd_camera">
         <pose>0 0 0 0 0 0</pose>
-        <gz_frame_id>camera_depth_optical_frame</gz_frame_id>
+        <gz_frame_id>${frame_id}</gz_frame_id>
         <always_on>true</always_on>
         <update_rate>15.0</update_rate>
         <visualize>true</visualize>
-        <topic>/camera_gz</topic>
+        <topic>${topic}</topic>
         <camera>
           <horizontal_fov>1.396</horizontal_fov>
@@ -53,5 +55,6 @@
     <joint name="gripper_controller"><command_interface name="position"/><state_interface name="position"/><state_interface name="velocity"/></joint>
   </xacro:macro>
-  <xacro:macro name="pro450_gz_ros2_control">
+  <xacro:macro name="pro450_gz_ros2_control"
+               params="root_link:='base_root' root_kinematic:='true'">
     <ros2_control name="Pro450GazeboSystem" type="system">
       <hardware>
@@ -60,5 +63,5 @@
       <xacro:pro450_arm_joint_interfaces/>
     </ros2_control>
-    <gazebo reference="base_root"><kinematic>true</kinematic></gazebo>
+    <gazebo reference="${root_link}"><kinematic>${root_kinematic}</kinematic></gazebo>
     <gazebo>
       <plugin filename="gz_ros2_control-system"

File: agbot/pro450_description/urdf/pro450_myagv_pro.urdf.xacro (robot description, xacro)
@@ -14,4 +14,8 @@
   <xacro:arg name="include_chassis_gz_camera" default="false"/>
   <xacro:arg name="include_wrist_camera" default="true"/>
+  <!-- MoveIt uses a stopped-base view of this model: wheel rotations are
+       irrelevant to arm planning and otherwise require unavailable wheel
+       joint states.  Gazebo/Nav2 keep the default continuous joints. -->
+  <xacro:arg name="planning_fixed_base" default="false"/>
   <!-- Deck mount for Pro450. Z matches the official top-deck height near laser_link. -->
   <xacro:arg name="arm_mount_x" default="0.0"/>
@@ -67,10 +71,19 @@
       </collision>
     </link>
-    <joint name="${name}_joint" type="continuous">
-      <parent link="base_link"/>
-      <child link="${name}_link"/>
-      <origin xyz="${x} ${y} ${z}" rpy="0 0 0"/>
-      <axis xyz="0 1 0"/>
-    </joint>
+    <xacro:if value="$(arg planning_fixed_base)">
+      <joint name="${name}_joint" type="fixed">
+        <parent link="base_link"/>
+        <child link="${name}_link"/>
+        <origin xyz="${x} ${y} ${z}" rpy="0 0 0"/>
+      </joint>
+    </xacro:if>
+    <xacro:unless value="$(arg planning_fixed_base)">
+      <joint name="${name}_joint" type="continuous">
+        <parent link="base_link"/>
+        <child link="${name}_link"/>
+        <origin xyz="${x} ${y} ${z}" rpy="0 0 0"/>
+        <axis xyz="0 1 0"/>
+      </joint>
+    </xacro:unless>
   </xacro:macro>
   <xacro:agv_wheel name="right_rear_wheel" mesh="wheel_rb_link.stl"
@@ -120,38 +133,41 @@
        Optical frames + optional Gazebo RGB-D for sim SLAM. -->
   <xacro:if value="$(arg include_chassis_orbbec)">
-    <link name="camera_link"/>
-    <joint name="camera_joint" type="fixed">
+    <link name="nav_camera_link"/>
+    <joint name="nav_camera_joint" type="fixed">
       <parent link="base_link"/>
-      <child link="camera_link"/>
+      <child link="nav_camera_link"/>
       <origin xyz="0.23191 0 0.14928" rpy="0 0 0"/>
     </joint>
     <!-- ROS optical convention: Z forward, X right, Y down -->
-    <link name="camera_depth_frame"/>
-    <joint name="camera_depth_joint" type="fixed">
-      <parent link="camera_link"/>
-      <child link="camera_depth_frame"/>
-      <origin xyz="0 0 0" rpy="0 0 0"/>
-    </joint>
-    <link name="camera_depth_optical_frame"/>
-    <joint name="camera_depth_optical_joint" type="fixed">
-      <parent link="camera_depth_frame"/>
-      <child link="camera_depth_optical_frame"/>
+    <link name="nav_camera_depth_frame"/>
+    <joint name="nav_camera_depth_joint" type="fixed">
+      <parent link="nav_camera_link"/>
+      <child link="nav_camera_depth_frame"/>
+      <origin xyz="0 0 0" rpy="0 0 0"/>
+    </joint>
+    <link name="nav_camera_depth_optical_frame"/>
+    <joint name="nav_camera_depth_optical_joint" type="fixed">
+      <parent link="nav_camera_depth_frame"/>
+      <child link="nav_camera_depth_optical_frame"/>
       <origin xyz="0 0 0" rpy="${-pi/2} 0 ${-pi/2}"/>
     </joint>
-    <link name="camera_color_frame"/>
-    <joint name="camera_color_joint" type="fixed">
-      <parent link="camera_link"/>
-      <child link="camera_color_frame"/>
-      <origin xyz="0 0 0" rpy="0 0 0"/>
-    </joint>
-    <link name="camera_color_optical_frame"/>
-    <joint name="camera_color_optical_joint" type="fixed">
-      <parent link="camera_color_frame"/>
-      <child link="camera_color_optical_frame"/>
+    <link name="nav_camera_color_frame"/>
+    <joint name="nav_camera_color_joint" type="fixed">
+      <parent link="nav_camera_link"/>
+      <child link="nav_camera_color_frame"/>
+      <origin xyz="0 0 0" rpy="0 0 0"/>
+    </joint>
+    <link name="nav_camera_color_optical_frame"/>
+    <joint name="nav_camera_color_optical_joint" type="fixed">
+      <parent link="nav_camera_color_frame"/>
+      <child link="nav_camera_color_optical_frame"/>
       <origin xyz="0 0 0" rpy="${-pi/2} 0 ${-pi/2}"/>
     </joint>
     <xacro:if value="$(arg include_chassis_gz_camera)">
       <xacro:include filename="$(find pro450_description)/urdf/pro450_gz_plugins.xacro"/>
-      <xacro:pro450_chassis_gz_rgbd_camera parent_link="camera_depth_frame" far="8.0"/>
+      <xacro:pro450_chassis_gz_rgbd_camera
+        parent_link="nav_camera_depth_frame" far="8.0"
+        topic="/nav_camera_gz"
+        frame_id="nav_camera_depth_optical_frame"/>
     </xacro:if>
   </xacro:if>
@@ -169,3 +185,20 @@
     <origin xyz="0 0 0" rpy="0 0 0"/>
   </joint>
+  <!-- Fortress drives the complete chassis+arm model as one rigid mobile
+       carrier while gz_ros2_control owns only the arm and gripper joints. -->
+  <xacro:if value="$(arg use_gz_control)">
+    <gazebo>
+      <plugin filename="ignition-gazebo-velocity-control-system"
+              name="gz::sim::systems::VelocityControl"/>
+      <plugin filename="ignition-gazebo-odometry-publisher-system"
+              name="gz::sim::systems::OdometryPublisher">
+        <odom_frame>odom</odom_frame>
+        <robot_base_frame>base_footprint</robot_base_frame>
+        <dimensions>2</dimensions>
+        <odom_publish_frequency>50</odom_publish_frequency>
+        <odom_topic>/model/pro450_myagv/odometry</odom_topic>
+        <tf_topic>/model/pro450_myagv/tf</tf_topic>
+      </plugin>
+    </gazebo>
+  </xacro:if>
 </robot>
